Commit message: feat: add Ouster lidar URDF and update DepthAI camera description

File: src/playground/urdf/depthai_camera_description.urdf.xacro (robot description, xacro)
@@ -1,21 +1,20 @@
 <?xml version="1.0"?>
 <robot name="depthai_camera" xmlns:xacro="http://ros.org/wiki/xacro">
-	<xacro:arg name="camera_name" default="oak" />
+	<xacro:arg name="camera_name"  default="oak" />
 	<xacro:arg name="camera_model" default="OAK-D" />
-	<xacro:arg name="base_frame" default="oak-d_frame" />
+	<xacro:arg name="base_frame"   default="oak-d_frame" />
 	<xacro:arg name="parent_frame" default="oak-d-base-frame" />
 	<xacro:arg name="cam_pos_x" default="0.0" />
 	<xacro:arg name="cam_pos_y" default="0.0" />
 	<xacro:arg name="cam_pos_z" default="0.0" />
-	<xacro:arg name="cam_roll" default="0.0" />
+	<xacro:arg name="cam_roll"  default="0.0" />
 	<xacro:arg name="cam_pitch" default="0.0" />
-	<xacro:arg name="cam_yaw" default="0.0" />
-	<xacro:arg name="rs_compat" default="false" />
+	<xacro:arg name="cam_yaw"   default="0.0" />
 	<xacro:include filename="$(find depthai_descriptions)/urdf/include/depthai_macro.urdf.xacro" />
 	<link name="$(arg parent_frame)" />
 	<xacro:depthai_camera camera_name="$(arg camera_name)" parent="$(arg parent_frame)"
 		camera_model="$(arg camera_model)" base_frame="$(arg base_frame)"
-		cam_pos_x="$(arg cam_pos_x)" cam_pos_y="$(arg cam_pos_y)" cam_pos_z="$(arg cam_pos_z)"
-		cam_roll="$(arg cam_roll)" cam_pitch="$(arg cam_pitch)" cam_yaw="$(arg cam_yaw)"
-		rs_compat="$(arg rs_compat)" />
+		cam_pos_x="$(arg cam_pos_x)"       cam_pos_y="$(arg cam_pos_y)" cam_pos_z="$(arg cam_pos_z)"
+		cam_roll="$(arg cam_roll)"         cam_pitch="$(arg cam_pitch)" cam_yaw="$(arg cam_yaw)"
+	/>
 </robot>

File: src/playground/urdf/depthai_camera_macro.urdf.xacro (robot description, xacro)
@@ -3,26 +3,21 @@
 	xmlns:xacro="http://ros.org/wiki/xacro">
 	<xacro:macro name="depthai_camera"
-		params="camera_name camera_model parent base_frame
-                                           cam_pos_x cam_pos_y cam_pos_z
-                                           cam_roll cam_pitch cam_yaw r:=0.8 g:=0.8 b:=0.8 a:=0.8 simulation:=false rs_compat:=false">
+		params="camera_name parent
+		camera_model base_frame
+        cam_pos_x cam_pos_y cam_pos_z
+        cam_roll cam_pitch cam_yaw
+		r:=0.8 g:=0.8 b:=0.8 a:=0.8
+		simulation:=false"
+		>
 		<xacro:include filename="$(find depthai_descriptions)/urdf/include/base_macro.urdf.xacro" />
-		<xacro:property name="M_PI" value="3.1415926535897931" />
-		<xacro:property name="model" value="${camera_model}" />
-		<xacro:property name="has_imu" value="false" />
+		<xacro:property name="M_PI" 	value="3.1415926535897931" />
+		<xacro:property name="model" 	value="${camera_model}" />
+		<xacro:property name="has_imu" 	value="false" />
 		<xacro:property name="baseline" value="0.075" />
-		<xacro:if value="${rs_compat}">
-			<xacro:property name="frame_suffix" value="frame" />
-			<xacro:property name="optical_frame_suffix" value="optical_frame" />
-			<xacro:property name="rgb_name" value="color" />
-			<xacro:property name="left_name" value="infra2" />
-			<xacro:property name="right_name" value="infra1" />
-		</xacro:if>
-		<xacro:unless value="${rs_compat}">
-			<xacro:property name="frame_suffix" value="camera_frame" />
-			<xacro:property name="optical_frame_suffix" value="camera_optical_frame" />
-			<xacro:property name="rgb_name" value="rgb" />
-			<xacro:property name="left_name" value="left" />
-			<xacro:property name="right_name" value="right" />
-		</xacro:unless>
+		<xacro:property name="frame_suffix" 		value="camera_frame" />
+		<xacro:property name="optical_frame_suffix" value="camera_optical_frame" />
+		<xacro:property name="rgb_name" 			value="rgb" />
+		<xacro:property name="left_name" 			value="left" />
+		<xacro:property name="right_name" 			value="right" />
 		<xacro:if value="${model in ['OAK-D-SR']}">
 			<xacro:property name="baseline" value="0.02" />
