Commit message: local: stuff

File: src/playground/urdf/sensor_mounts.urdf.xacro (robot description, xacro)
@@ -1,59 +1,59 @@
 <?xml version="1.0"?>
 <robot name="multi_sensor_robot" xmlns:xacro="http://www.ros.org/wiki/xacro">
-  <link name="base-link"/>
-  <link name="mount-link"/>
-  <joint name="mount-link-joint" type="revolute">
-    <parent link="base-link"/>
-    <child link="mount-link"/>
+  <link name="base_link"/>
+  <link name="mount_link"/>
+  <joint name="mount_link_joint" type="revolute">
+    <parent link="base_link"/>
+    <child link="mount_link"/>
     <origin xyz="-0.27 0.0 0.0" rpy="0 0 0"/>
     <axis xyz="0 0 1"/>
     <limit effort="5" velocity="1.0" lower="-3.14" upper="3.14"/>
   </joint>
-  <link name="sensor-mount-00-link"/>
-  <joint name="sensor-mount-00-joint" type="revolute">
-    <parent link="mount-link"/>
-    <child link="sensor-mount-00-link"/>
+  <link name="sensor_mount_00_link"/>
+  <joint name="sensor_mount_00_joint" type="revolute">
+    <parent link="mount_link"/>
+    <child link="sensor_mount_00_link"/>
     <origin xyz="-0.12 0.0 0.22" rpy="0 0 3.14159265359"/>
     <axis xyz="0 0 1"/>
     <limit effort="5" velocity="1.0" lower="-3.14" upper="3.14"/>
   </joint>
-  <link name="sensor-mount-01-link"/>
-  <joint name="sensor-mount-01-joint" type="revolute">
-    <parent link="mount-link"/>
-    <child link="sensor-mount-01-link"/>
+  <link name="sensor_mount_01_link"/>
+  <joint name="sensor_mount_01_joint" type="revolute">
+    <parent link="mount_link"/>
+    <child link="sensor_mount_01_link"/>
     <origin xyz="-0.12 0.0 0.12" rpy="0 0 3.14159265359"/>
     <axis xyz="0 0 1"/>
     <limit effort="5" velocity="1.0" lower="-3.14" upper="3.14"/>
   </joint>
-  <link name="sensor-mount-02-link"/>
-  <joint name="sensor-mount-02-joint" type="revolute">
-    <parent link="mount-link"/>
-    <child link="sensor-mount-02-link"/>
+  <link name="sensor_mount_02_link"/>
+  <joint name="sensor_mount_02_joint" type="revolute">
+    <parent link="mount_link"/>
+    <child link="sensor_mount_02_link"/>
     <origin xyz="-0.05 0.0 0.3" rpy="0 0 0"/>
     <axis xyz="0 0 1"/>
     <limit effort="5" velocity="1.0" lower="-3.14" upper="3.14"/>
   </joint>
-  <link name="ouster-os-link"/>
-  <joint name="ouster-os-joint" type="fixed">
-    <parent link="sensor-mount-02-link"/>
-    <child link="ouster-os-link"/>
+  <link name="lidar_00_link"/>
+  <joint name="ouster_os_joint" type="fixed">
+    <parent link="sensor_mount_02_link"/>
+    <child link="lidar_00_link"/>
     <origin xyz="0 0 0" rpy="0 -0.2618 0"/>
   </joint>
-  <link name="lidar"/>
-  <joint name="ouster-lidar-joint" type="fixed">
-    <parent link="ouster-os-link"/>
-    <child link="lidar"/>
+  <link name="lidar_00_lidar_frame"/>
+  <joint name="ouster_lidar_joint" type="fixed">
+    <parent link="lidar_00_link"/>
+    <child link="lidar_00_lidar_frame"/>
   <origin xyz="0 0 0" rpy="0 0 0"/>
   </joint>
-  <link name="imu"/>
-  <joint name="ouster-imu-joint" type="fixed">
-    <parent link="ouster-os-link"/>
-    <child link="imu"/>
+  <link name="lidar_00_imu_frame"/>
+  <joint name="ouster_imu_joint" type="fixed">
+    <parent link="lidar_00_link"/>
+    <child link="lidar_00_imu_frame"/>
   <origin xyz="0 0 0" rpy="0 0 0"/>
   </joint>
-  <!-- <link name="sensor-mount-03-link"/>
-  <joint name="sensor-mount-03-joint" type="revolute">
-    <parent link="mount-link"/>
-    <child link="sensor-mount-03-link"/>
+  <!-- <link name="sensor_mount_03_link"/>
+  <joint name="sensor_mount_03_joint" type="revolute">
+    <parent link="mount_link"/>
+    <child link="sensor_mount_03_link"/>
     <origin xyz="0.0 0.0 0.0" rpy="0 0 0"/>
     <axis xyz="0 0 1"/>
