Commit message: feat: add mapping configuration

File: src/rover_autonomy/urdf/camera.urdf.xacro (robot description, xacro)
@@ -12,4 +12,16 @@
         </joint>
         <link name="${camera_name}_link">
+            <visual>
+                <origin xyz="0.00 -0.048 0.02" rpy="1.5708 0 1.5708"/>
+                <geometry>
+                    <mesh filename="package://rover_autonomy/mesh/oak_d_pro_w_poe.stl" scale="0.001 0.001 0.001"/>
+                </geometry>
+            </visual>
+            <collision>
+                <origin xyz="0 0 0" rpy="0 0 0" />
+                <geometry>
+                    <box size="0.03 0.10 0.03"/>
+                </geometry>
+            </collision>
         </link>
         <link name="${camera_name}_model_origin" />

File: src/rover_autonomy/urdf/lidar.urdf.xacro (robot description, xacro)
@@ -12,4 +12,16 @@
         </joint>
         <link name="${lidar_name}_link">
+            <visual>
+                <origin xyz="0 0 0" rpy="0 0 0" />
+                <geometry>
+                    <mesh filename="package://rover_autonomy/mesh/ouster_os1.dae" scale="1.0 1.0 1.0"/>
+                </geometry>
+            </visual>
+            <collision>
+                <origin xyz="0 0 0" rpy="0 0 0" />
+                <geometry>
+                    <box size="0.03 0.10 0.03"/>
+                </geometry>
+            </collision>
         </link>
         <link name="${lidar_name}_model_origin" />

File: src/rover_autonomy/urdf/sensor_mounts.urdf.xacro (robot description, xacro)
@@ -20,10 +20,10 @@
     <origin xyz="-0.12 0.0 0.12" rpy="0 0 3.14159265359"/>
   </joint>
-  <link name="sensor_mount_02_link"/>
+  <!-- <link name="sensor_mount_02_link"/>
   <joint name="sensor_mount_02_joint" type="fixed">
     <parent link="mount_link"/>
     <child link="sensor_mount_02_link"/>
     <origin xyz="-0.05 0.0 0.3" rpy="0 0 0"/>
-  </joint>
+  </joint> -->
   <!-- <link name="sensor_mount_03_link"/>
   <joint name="sensor_mount_03_joint" type="fixed">
